Commit message: use xacro instead of direct urdf

File: src/my_robot_description/urdf/arm.xacro (robot description, xacro)
@@ -1,10 +1,4 @@
 <?xml version="1.0" ?>
-<robot name="my_robot">
-    <material name="grey">
-        <color rgba="0.5 0.5 0.5 1" />
-    </material>
-    <material name="blue">
-        <color rgba="0 0 0.5 1" />
-    </material>
+<robot xmlns:xacro="http://www.ros.org/wiki/xacro">
     <!-- LINKS -->
     <link name="base_link">

Commit message: add collision geometries for robot arm links

File: src/my_robot_description/urdf/arm.xacro (robot description, xacro)
@@ -10,4 +10,10 @@
             <material name="grey" />
         </visual>
+        <collision>
+            <geometry>
+                <box size="0.4 0.4 0.1" />
+            </geometry>
+            <origin xyz="0 0 0.05" rpy="0 0 0" />
+        </collision>
     </link>
     <link name="shoulder_link">
@@ -19,4 +25,10 @@
             <material name="blue" />
         </visual>
+        <collision>
+            <geometry>
+                <cylinder length="0.5" radius="0.1" />
+            </geometry>
+            <origin xyz="0 0 0.25" rpy="0 0 0" />
+        </collision>
     </link>
     <link name="arm_link">
@@ -28,4 +40,10 @@
             <material name="grey" />
         </visual>
+        <collision>
+        <geometry>
+            <cylinder length="0.6" radius="0.05" />
+        </geometry>
+        <origin xyz="0 0 0.3" rpy="0 0 0" />
+        </collision>
     </link>
     <link name="elbow_link">
@@ -37,4 +55,10 @@
             <material name="blue" />
         </visual>
+        <collision>
+        <geometry>
+            <cylinder length="0.1" radius="0.05" />
+        </geometry>
+        <origin xyz="0 0 0.05" rpy="0 0 0" />
+        </collision>
     </link>
     <link name="forearm_link">
@@ -46,4 +70,10 @@
             <material name="grey" />
         </visual>
+        <collision>
+        <geometry>
+            <cylinder length="0.5" radius="0.05" />
+        </geometry>
+        <origin xyz="0 0 0.25" rpy="0 0 0" />
+        </collision>
     </link>
     <link name="wrist_link">
@@ -55,4 +85,10 @@
             <material name="blue" />
         </visual>
+        <collision>
+        <geometry>
+            <box size="0.1 0.1 0.05" />
+        </geometry>
+        <origin xyz="0 0 0.025" rpy="0 0 0" />
+        </collision>
     </link>
     <link name="hand_link">
@@ -64,4 +100,10 @@
             <material name="grey" />
         </visual>
+        <collision>
+        <geometry>
+            <box size="0.1 0.1 0.02" />
+        </geometry>
+        <origin xyz="0 0 0.01" rpy="0 0 0" />
+        </collision>
     </link>
     <link name="tool_link" />
